File: prototype/pcb/$watch_proto_pcb.sch (KiCad schematic (older format))
At the start: 3 parts, among them P3 CONN_01X04

Commit message: Added concentric power traces
Parts:
- gave numbers to parts that had none: 2
Changed lines of the file:
@@
 BLANK
 $Comp
-L PWR_FLAG #FLG04
+L PWR_FLAG #FLG03
 U 1 1 574F2A39
 P 4550 3950
-F 0 "#FLG04" H 4550 4045 50  0001 C CNN
+F 0 "#FLG03" H 4550 4045 50  0001 C CNN
 F 1 "PWR_FLAG" H 4550 4130 50  0000 C CNN
 F 2 "" H 4550 3950 60  0000 C CNN
@@
 Connection ~ 4550 4150
 $Comp
-L PWR_FLAG #FLG05
+L PWR_FLAG #FLG04
 U 1 1 574F2A91
 P 4550 4750
-F 0 "#FLG05" H 4550 4845 50  0001 C CNN
+F 0 "#FLG04" H 4550 4845 50  0001 C CNN
 F 1 "PWR_FLAG" H 4550 4930 50  0000 C CNN
 F 2 "" H 4550 4750 60  0000 C CNN
@@
 	6950 5400 7650 5400
 $Comp
-L CONN_01X06 P?
+L CONN_01X06 P2
 U 1 1 5751DBAE
 P 3700 4400
-F 0 "P?" H 3700 4750 50  0000 C CNN
+F 0 "P2" H 3700 4750 50  0000 C CNN
 F 1 "CONN_01X06" V 3800 4400 50  0000 C CNN
 F 2 "Pin_Headers:Pin_Header_Straight_1x06" H 3700 4400 60  0001 C CNN
@@
 $EndComp
 $Comp
-L CONN_01X04 P?
+L CONN_01X04 P1
 U 1 1 5751DC25
 P 7850 4300
-F 0 "P?" H 7850 4550 50  0000 C CNN
+F 0 "P1" H 7850 4550 50  0000 C CNN
 F 1 "CONN_01X04" V 7950 4300 50  0000 C CNN
 F 2 "Pin_Headers:Pin_Header_Straight_1x04" H 7850 4300 60  0001 C CNN
